File: KiCad/upduinov2.1-SRAM/upduinov2.1-SRAM.kicad_pcb (KiCad board)
At the start: 2 copper layers, 50 x 22.9 mm, 5 parts, among them J6 77311-801-02LF, J8 1p-2.54, J9 1p-2.54

Commit message: fixed pin number on upd-SRAM pcb
Other:
- board text added: "36"
Changed lines of the file:
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@@
     (effects (font (size 0.77216 0.77216) (thickness 0.097536)) (justify left bottom))
   )
-  (gr_text 35 (at 132.595581 136.271) (layer F.SilkS)
+  (gr_text 36 (at 132.595581 136.271) (layer F.SilkS)
     (effects (font (size 0.77216 0.77216) (thickness 0.097536)) (justify left bottom))
   )

Commit message: New Upduino shield
Parts:
- removed J6: 77311-801-02LF, upduino_v2.1_release:1X02
- removed J8, J9: 1p-2.54, upduino_v2.1_release:1P-65_35MIL
- removed JP5, JP6: M161X16_NO_SILK, upduino_v2.1_release:1X16_NO_SILK
Other:
- board outline removed
- board text removed: "1"
- board text removed: "11"
- board text removed: "12"
- board text removed: "13"
- board text removed: "18"
- board text removed: "19"
- board text removed: "2"
- board text removed: "21"
- board text removed: "23"
- board text removed: "25"
- board text removed: "26"
- board text removed: "27"
- board text removed: "28"
- board text removed: "3"
- board text removed: "3.3V"
- board text removed: "31"
- board text removed: "32"
- board text removed: "34"
- board text removed: "35"
- board text removed: "36"
- board text removed: "37"
- board text removed: "38"
- board text removed: "4"
- board text removed: "42"
- board text removed: "43"
- board text removed: "44"
- board text removed: "45"
- board text removed: "46"
- board text removed: "47"
- board text removed: "48"
- board text removed: "5V"
- board text removed: "6"
- board text removed: "9"
- board text removed: "GND"

Commit message: updv2 pcb v1 w handroute decoupler
Parts:
- added C1: 0.1uF, Capacitor_SMD:C_0805_2012Metric, F.Cu at (160.0, 105.4)
- added J1: Conn_01x16_Male, Connector_PinHeader_2.54mm:PinHeader_1x16_P2.54mm_Vertical, F.Cu at (152.4, 101.6)
- added J2: Conn_01x18_Male, Connector_PinHeader_2.54mm:PinHeader_1x18_P2.54mm_Vertical, F.Cu at (170.2, 96.5)
- added U1: CY62157, Package_SO:TSOP-I-48_18.4x12mm_P0.5mm, F.Cu at (161.3, 118.1)
Routing:
- net /A16: track 0.00 -> 35.9 mm
- net /A15: track 0.00 -> 35.6 mm
- net +3V3: track 0.00 -> 34.9 mm
- net /A19: track 0.00 -> 28.0 mm
- net /D1: track 0.00 -> 25.9 mm
- net /A1: track 0.00 -> 25.1 mm
- net /A2: track 0.00 -> 24.8 mm
- net /~OE: track 0.00 -> 24.2 mm, vias 0 -> 1
- net /A3: track 0.00 -> 23.3 mm
- net /A4: track 0.00 -> 21.8 mm
- net /D4: track 0.00 -> 20.6 mm
- net /A5: track 0.00 -> 20.2 mm
- net /D7: track 0.00 -> 19.8 mm
- net /A14: track 0.00 -> 19.7 mm, vias 0 -> 1
- net /A6: track 0.00 -> 18.7 mm
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- added copper zone on B.Cu, net GND
Other:
- board outline added: 25.4 x 50.8 mm
- board text added: "+3.3V"
- board text added: "10"
- board text added: "A0"
- board text added: "A1"
- board text added: "A11"
- board text added: "A12"
- board text added: "A13"
- board text added: "A14"
- board text added: "A15"
- board text added: "A16"
- board text added: "A17"
- board text added: "A18"
- board text added: "A19"
- board text added: "A2"
- board text added: "A3"
- board text added: "A4"
- board text added: "A5"
- board text added: "A6"
- board text added: "A7"
- board text added: "A8"
- board text added: "A9"
- board text added: "D0"
- board text added: "D1"
- board text added: "D2"
- board text added: "D3"
- board text added: "D4"
- board text added: "D5"
- board text added: "D6"
- board text added: "D7"
- board text added: "GND"
- board text added: "NC"
- board text added: "SamWibatt 2019"
- board text added: "Upduino v2 SRAM Adapter 1Mx8 CY62157EV30"
- board text added: "~OE"
- board text added: "~WE"

Commit message: added board version number
Other:
- board text added: "Board v1"
Changed lines of the file:
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@@
   (general
     (thickness 1.6)
-    (drawings 40)
+    (drawings 41)
     (tracks 257)
     (zones 0)
@@
   (layers
     (0 F.Cu signal)
-    (31 B.Cu signal hide)
+    (31 B.Cu signal)
     (34 B.Paste user)
     (35 F.Paste user)
@@
     )
   )
+  (gr_text "Board v1" (at 159.2 99.7) (layer F.SilkS)
+    (effects (font (size 1 1) (thickness 0.15)))
+  )
   (gr_text "SamWibatt\n2019" (at 161.29 138.43) (layer F.SilkS)
